File: crossing/crossing.kicad_sch (KiCad schematic)
At the start: 17 parts, among them J1 PAD, Q2 2N3904, Q3 2N3904, SW1 SW_SPDT

Commit message: Another WIP
Parts:
- D1, D2: footprint LED_THT:LED_D10.0mm -> lib:LED_D10.0mm
Changed lines of the file:
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@@
 			)
 		)
-		(property "Footprint" "LED_THT:LED_D10.0mm"
+		(property "Footprint" "lib:LED_D10.0mm"
 			(at 117.475 91.44 0)
 			(effects
@@
 			)
 		)
-		(property "Footprint" "LED_THT:LED_D10.0mm"
+		(property "Footprint" "lib:LED_D10.0mm"
 			(at 173.355 91.44 0)
 			(effects

Commit message: Init new branch + development
Parts:
- BT1: footprint kit-fp:CONNFLY_DS1092-04 -> lib:CONNFLY_DS1092-04
- C1: footprint kit-fp:CP_Radial_D6.3mm_P2.50mm+SMD_0805 -> lib:CP_Radial_D6.3mm_P2.50mm+SMD_0805
- J1: footprint kit-fp:Touchpad_resistive -> lib:Touchpad_resistive
- Q2, Q3: footprint kit-fp:TO-92L_Inline_Wide+SMD_SOT-23 -> lib:TO-92L_Inline_Wide+SMD_SOT-23
- R11, R12, R3, R4: footprint kit-fp:R_Axial_SMD_DIN0207_L6.3mm_D2.5mm_P10.16mm_Horizontal -> lib:R_Axial_SMD_DIN0207_L6.3mm_D2.5mm_P10.16mm_Horizontal
Changed lines of the file:
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@@
 			)
 		)
-		(property "Footprint" "kit-fp:R_Axial_SMD_DIN0207_L6.3mm_D2.5mm_P10.16mm_Horizontal"
+		(property "Footprint" "lib:R_Axial_SMD_DIN0207_L6.3mm_D2.5mm_P10.16mm_Horizontal"
 			(at 160.147 82.55 90)
 			(effects
@@
 			)
 		)
-		(property "Footprint" "kit-fp:R_Axial_SMD_DIN0207_L6.3mm_D2.5mm_P10.16mm_Horizontal"
+		(property "Footprint" "lib:R_Axial_SMD_DIN0207_L6.3mm_D2.5mm_P10.16mm_Horizontal"
 			(at 119.253 82.55 90)
 			(effects
@@
 			)
 		)
-		(property "Footprint" "kit-fp:CONNFLY_DS1092-04"
+		(property "Footprint" "lib:CONNFLY_DS1092-04"
 			(at 102.235 102.616 90)
 			(effects
@@
 			)
 		)
-		(property "Footprint" "kit-fp:Touchpad_resistive"
+		(property "Footprint" "lib:Touchpad_resistive"
 			(at 149.225 81.28 0)
 			(effects
@@
 			)
 		)
-		(property "Footprint" "kit-fp:TO-92L_Inline_Wide+SMD_SOT-23"
+		(property "Footprint" "lib:TO-92L_Inline_Wide+SMD_SOT-23"
 			(at 114.935 108.585 0)
 			(effects
@@
 			)
 		)
-		(property "Footprint" "kit-fp:R_Axial_SMD_DIN0207_L6.3mm_D2.5mm_P10.16mm_Horizontal"
+		(property "Footprint" "lib:R_Axial_SMD_DIN0207_L6.3mm_D2.5mm_P10.16mm_Horizontal"
 			(at 149.225 93.218 90)
 			(effects
@@
 			)
 		)
-		(property "Footprint" "kit-fp:R_Axial_SMD_DIN0207_L6.3mm_D2.5mm_P10.16mm_Horizontal"
+		(property "Footprint" "lib:R_Axial_SMD_DIN0207_L6.3mm_D2.5mm_P10.16mm_Horizontal"
 			(at 139.065 93.218 90)
 			(effects
@@
 			)
 		)
-		(property "Footprint" "kit-fp:R_Axial_SMD_DIN0207_L6.3mm_D2.5mm_P10.16mm_Horizontal"
+		(property "Footprint" "lib:R_Axial_SMD_DIN0207_L6.3mm_D2.5mm_P10.16mm_Horizontal"
 			(at 130.683 82.55 90)
 			(effects
@@
 			)
 		)
-		(property "Footprint" "kit-fp:TO-92L_Inline_Wide+SMD_SOT-23"
+		(property "Footprint" "lib:TO-92L_Inline_Wide+SMD_SOT-23"
 			(at 175.895 108.585 0)
 			(effects
@@
 			)
 		)
-		(property "Footprint" "kit-fp:R_Axial_SMD_DIN0207_L6.3mm_D2.5mm_P10.16mm_Horizontal"
+		(property "Footprint" "lib:R_Axial_SMD_DIN0207_L6.3mm_D2.5mm_P10.16mm_Horizontal"
 			(at 171.577 82.55 90)
 			(effects
@@
 			)
 		)
-		(property "Footprint" "kit-fp:CP_Radial_D6.3mm_P2.50mm+SMD_0805"
+		(property "Footprint" "lib:CP_Radial_D6.3mm_P2.50mm+SMD_0805"
 			(at 127.635 98.0948 0)
 			(effects
@@
 			)
 		)
-		(property "Footprint" "kit-fp:CP_Radial_D6.3mm_P2.50mm+SMD_0805"
+		(property "Footprint" "lib:CP_Radial_D6.3mm_P2.50mm+SMD_0805"
 			(at 163.195 100.0252 0)
 			(effects
