File: crossing/crossing.kicad_pcb (KiCad board)
At the start: 2 copper layers, 38 x 66.7 mm, 18 parts, among them J1 PAD, Q1 2N3904, Q2 2N3904, SW1 SW_SPDT

Commit message: Another WIP
Parts:
- D1, D2: footprint LED_THT:LED_D10.0mm -> lib:LED_D10.0mm
Other:
- board text removed: "logo was here"

Commit message: Init new branch + development
Parts:
- BT1: footprint kit-fp:CONNFLY_DS1092-04 -> lib:CONNFLY_DS1092-04
- C1, C2: footprint kit-fp:CP_Radial_D6.3mm_P2.50mm+SMD_0805 -> lib:CP_Radial_D6.3mm_P2.50mm+SMD_0805
- J1: footprint kit-fp:Touchpad_resistive -> lib:Touchpad_resistive
- Q1, Q2: footprint kit-fp:TO-92L_Inline_Wide+SMD_SOT-23 -> lib:TO-92L_Inline_Wide+SMD_SOT-23
- R1, R2, R3, R4, R5, R6: footprint kit-fp:R_Axial_SMD_DIN0207_L6.3mm_D2.5mm_P10.16mm_Horizontal -> lib:R_Axial_SMD_DIN0207_L6.3mm_D2.5mm_P10.16mm_Horizontal
Other:
- outline, holes or cut-outs redrawn
