File: bat/bat.kicad_sch (KiCad schematic)
At the start: 16 parts, among them Q1 2N3904, Q2 2N3904, Q3 2N3904, SW1 SW_SPDT

Commit message: boom prask netopyr netopyr
Parts:
- removed Q3: 2N3904, Package_TO_SOT_THT:TO-92L_Inline_Wide, symbol Transistor_BJT:2N3904
- added Q3: S8550, Package_TO_SOT_THT:TO-92L_Inline_Wide, symbol Transistor_BJT:S8550
- R1, R2: value 10k -> 68k
- R3, R4: value 47k -> 100k
- R5: value 330 -> 47R
- R6: value 300k -> 47k
Connections:
- net GND: now also Q3.3 (C)
- net at C3.1, R6.2: now also Q3.2 (B)
- net at D1.1 (K), D2.1 (K): now also Q3.1 (E)

Commit message: netopyr
Other:
- note added: "V2.0"
- moved on the sheet: BT1, C1, C2, C3, D1, D2, Q1, Q2, Q3, R1, R2, R3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
