File: trafficlight/pcb_2032/trafficlight.kicad_pcb (KiCad board)
At the start: 2 copper layers, 10 x 30 mm, 10 parts, among them SW1 SW_Push, U1 PIC10F322-IOT

Commit message: Added cat-pin, bat, traffic light?
Parts:
- moved D1 0.25 mm to (137.0, 99.5)
- moved R3 0.15 mm to (137.0, 101.6)
Routing:
- net /LED_R: track 30.2 -> 28.9 mm
- net /BUTTON: track 11.7 -> 12.3 mm
Other:
- board text removed: "03:27"
