File: cat-pin/cat-pin.kicad_pcb (KiCad board)
At the start: 2 copper layers, 36.2 x 26.9 mm, 0 parts

Commit message: Production version
Other:
- board size 36.2 x 26.9 mm -> 33.9 x 27.1 mm
- board text removed: "adam@pajecistavebnice.cz"
