File: heart-badge/heart-badge.kicad_pcb (KiCad board)
At the start: 2 copper layers, 37 x 32.6 mm, 17 parts

Commit message: heart-badge development
Parts:
- added REF**: MS-22D28-G020, lib:MS-22D28-G020, F.Cu at (121.5, 64.0)
Changed lines of the file:
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@@
 		)
 	)
+	(footprint "lib:MS-22D28-G020"
+		(layer "F.Cu")
+		(at 121.5 64)
+		(property "Reference" "REF**"
+			(at 0 -6.5 0)
+			(unlocked yes)
+			(layer "F.SilkS")
+			(effects
+				(font
+					(size 1 1)
+					(thickness 0.15)
+				)
+			)
+		)
+		(property "Value" "MS-22D28-G020"
+			(at 0 1 0)
+			(unlocked yes)
+			(layer "F.Fab")
+			(effects
+				(font
+					(size 1 1)
+					(thickness 0.15)
+				)
+			)
+		)
+		(property "Footprint" "lib:MS-22D28-G020"
+			(at 0 0 0)
+			(unlocked yes)
+			(layer "F.Fab")
+			(hide yes)
+			(effects
+				(font
+					(size 1 1)
+					(thickness 0.15)
+				)
+			)
+		)
+		(property "Datasheet" ""
+			(at 0 0 0)
+			(unlocked yes)
+			(layer "F.Fab")
+			(hide yes)
+			(effects
+				(font
+					(size 1 1)
+					(thickness 0.15)
+				)
+			)
+		)
+		(property "Description" ""
+			(at 0 0 0)
+			(unlocked yes)
+			(layer "F.Fab")
+			(hide yes)
+			(effects
+				(font
+					(size 1 1)
+					(thickness 0.15)
+				)
+			)
+		)
+		(attr smd)
+		(fp_line
+			(start -3.5 -2)
+			(end -3.5 2)
+			(stroke
+				(width 0.12)
+				(type default)
+			)
+			(layer "F.SilkS")
+		)
+		(fp_line
+			(start -3.5 2)
+			(end 3.5 2)
+			(stroke
+				(width 0.12)
+				(type default)
+			)
+			(layer "F.SilkS")
+		)
+		(fp_line
+			(start -1.4 -0.75)
+			(end -1.4 0.7)
+			(stroke
+				(width 0.12)
+				(type default)
+			)
+			(layer "F.SilkS")
+		)
+		(fp_line
+			(start -1.4 -0.75)
+			(end 0 -0.75)
+			(stroke
+				(width 0.12)
+				(type default)
+			)
+			(layer "F.SilkS")
+		)
+		(fp_line
+			(start 0 0.7)
+			(end -1.4 0.7)
+			(stroke
+				(width 0.12)
+				(type default)
+			)
+			(layer "F.SilkS")
+		)
+		(fp_line
+			(start 3.5 -2)
+			(end -3.5 -2)
+			(stroke
+				(width 0.12)
+				(type default)
+			)
+			(layer "F.SilkS")
+		)
+		(fp_line
+			(start 3.5 2)
+			(end 3.5 -2)
+			(stroke
+				(width 0.12)
+				(type default)
+			)
+			(layer "F.SilkS")
+		)
+		(fp_rect
+			(start 0 -0.75)
+			(end 1.4 0.7)
+			(stroke
+				(width 0.12)
+				(type solid)
+			)
+			(fill solid)
+			(layer "F.SilkS")
+		)
+		(fp_rect
+			(start -4.25 -5.5)
+			(end 4.25 5.5)
+			(stroke
+				(width 0.12)
+				(type default)
+			)
+			(fill none)
+			(layer "Margin")
+		)
+		(fp_text user "${REFERENCE}"
+			(at 0 2.5 0)
+			(unlocked yes)
+			(layer "F.Fab")
+			(effects
+				(font
+					(size 1 1)
+					(thickness 0.15)
+				)
+			)
+		)
+		(pad "" np_thru_hole circle
+			(at -2.25 0 90)
+			(size 1.1 1.1)
+			(drill 1.1)
+			(layers "F&B.Cu" "*.Mask")
+		)
+		(pad "" np_thru_hole circle
+			(at 2.25 0 90)
+			(size 1.1 1.1)
+			(drill 1.1)
+			(layers "F&B.Cu" "*.Mask")
+		)
+		(pad "1" smd roundrect
+			(at -2 3.5 90)
+			(size 2.8 1.2)
+			(layers "F.Cu" "F.Paste" "F.Mask")
+			(roundrect_rratio 0.25)
+			(thermal_bridge_angle 45)
+		)
+		(pad "2" smd roundrect
+			(at 0 3.5 90)
+			(size 2.8 1.2)
+			(layers "F.Cu" "F.Paste" "F.Mask")
+			(roundrect_rratio 0.25)
+			(thermal_bridge_angle 45)
+		)
+		(pad "3" smd roundrect
+			(at 2 3.5 90)
+			(size 2.8 1.2)
+			(layers "F.Cu" "F.Paste" "F.Mask")
+			(roundrect_rratio 0.25)
+			(thermal_bridge_angle 45)
+		)
+		(pad "4" smd roundrect
+			(at 2 -3.5 90)
+			(size 2.8 1.2)
+			(layers "F.Cu" "F.Paste" "F.Mask")
+			(roundrect_rratio 0.25)
+			(thermal_bridge_angle 45)
+		)
+		(pad "5" smd roundrect
+			(at 0 -3.5 90)
+			(size 2.8 1.2)
+			(layers "F.Cu" "F.Paste" "F.Mask")
+			(roundrect_rratio 0.25)
+			(thermal_bridge_angle 45)
+		)
+		(pad "6" smd roundrect
+			(at -2 -3.5 90)
+			(size 2.8 1.2)
+			(layers "F.Cu" "F.Paste" "F.Mask")
+			(roundrect_rratio 0.25)
+			(thermal_bridge_angle 45)
+		)
+	)
 	(footprint "LED_SMD:LED_0805_2012Metric_Pad1.15x1.40mm_HandSolder"
 		(layer "F.Cu")
@@
 	)
 	(gr_poly
-		(pts
-			(xy 126.282486 66.232233) (xy 131.232233 61.282485) (xy 135.474873 65.525127) (xy 130.525127 70.474873)
-		)
-		(stroke
-			(width 0.1)
-			(type default)
-		)
-		(fill none)
-		(layer "Dwgs.User")
-	)
-	(gr_poly

Commit message: another one
Parts:
- removed REF** (x15): LED_0805_2012Metric_Pad1.15x1.40mm_HandSolder, LED_SMD:LED_0805_2012Metric_Pad1.15x1.40mm_HandSolder
- removed REF**: CR2032_SMD, lib:CR2032_SMD
- removed REF**: SW_JS202011SCQN, lib:SW_JS202011SCQN
- removed REF**: MS-22D28-G020, lib:MS-22D28-G020
- added BT1: Battery_Cell, lib:CR2032_SMD, B.Cu at (143.0, 77.0)
- added D1: LED, LED_SMD:LED_0805_2012Metric_Pad1.15x1.40mm_HandSolder, F.Cu at (143.0, 87.5)
- added D10: LED, LED_SMD:LED_0805_2012Metric_Pad1.15x1.40mm_HandSolder, F.Cu at (151.0, 62.5)
- added D11: LED, LED_SMD:LED_0805_2012Metric_Pad1.15x1.40mm_HandSolder, F.Cu at (156.5, 64.5)
- added D12: LED, LED_SMD:LED_0805_2012Metric_Pad1.15x1.40mm_HandSolder, F.Cu at (158.5, 70.0)
- added D13: LED, LED_SMD:LED_0805_2012Metric_Pad1.15x1.40mm_HandSolder, F.Cu at (156.0, 75.5)
- added D14: LED, LED_SMD:LED_0805_2012Metric_Pad1.15x1.40mm_HandSolder, F.Cu at (151.8, 79.8)
- added D15: LED, LED_SMD:LED_0805_2012Metric_Pad1.15x1.40mm_HandSolder, F.Cu at (147.5, 84.0)
- added D2: LED, LED_SMD:LED_0805_2012Metric_Pad1.15x1.40mm_HandSolder, F.Cu at (138.5, 84.0)
- added D3: LED, LED_SMD:LED_0805_2012Metric_Pad1.15x1.40mm_HandSolder, F.Cu at (134.2, 79.8)
- added D4: LED, LED_SMD:LED_0805_2012Metric_Pad1.15x1.40mm_HandSolder, F.Cu at (130.0, 75.5)
- added D5: LED, LED_SMD:LED_0805_2012Metric_Pad1.15x1.40mm_HandSolder, F.Cu at (127.5, 70.0)
- added D6: LED, LED_SMD:LED_0805_2012Metric_Pad1.15x1.40mm_HandSolder, F.Cu at (129.5, 64.5)
- added D7: LED, LED_SMD:LED_0805_2012Metric_Pad1.15x1.40mm_HandSolder, F.Cu at (135.0, 62.5)
- added D8: LED, LED_SMD:LED_0805_2012Metric_Pad1.15x1.40mm_HandSolder, F.Cu at (139.5, 65.0)
- added D9: LED, LED_SMD:LED_0805_2012Metric_Pad1.15x1.40mm_HandSolder, F.Cu at (146.5, 65.0)
- added R1: 200R, Resistor_SMD:R_0805_2012Metric_Pad1.20x1.40mm_HandSolder, B.Cu at (132.0, 66.5)
- added SW1: MST22D18G2, lib:SW_JS202011SCQN, B.Cu at (154.0, 66.5)
Routing:
- net Net-(D1-A): track 0.00 -> 141.5 mm, vias 0 -> 1
- net Net-(D1-K): track 0.00 -> 120.9 mm, vias 0 -> 1
- net Net-(BT1-+): track 0.00 -> 45.9 mm
- net Net-(BT1--): track 0.00 -> 16.1 mm
- added copper zone on B.Cu, net (none)
- added copper zone on F.Cu, net (none)
Other:
- board text added: "JLCJLCJLCJLC"
- board text added: "github.com/polaracep"

Commit message: Work work work
Routing:
- net Net-(D1-K): track 120.9 -> 122.3 mm
- net Net-(D1-A): track 141.5 -> 142.4 mm
Other:
- board text removed: "JLCJLCJLCJLC"
Changed lines of the file:
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@@
 		(layer "Edge.Cuts")
-	)
-	(gr_text "JLCJLCJLCJLC"
-		(at 143 86.25 0)
-		(layer "B.SilkS")
-		(effects
-			(font
-				(size 1 1)
-				(thickness 0.15)
-			)
-			(justify bottom mirror)
-		)
 	)
 	(gr_text "github.com/polaracep"
@@
 		(start 131.292893 67.292893)
 		(end 141 77)
-		(width 0.25)
+		(width 0.4)
 		(layer "B.Cu")
 		(net 1)
@@
 		(start 141 77)
 		(end 143 77)
-		(width 0.25)
+		(width 0.4)
 		(layer "B.Cu")
 		(net 1)
@@
 		(start 131.292893 67.207107)
 		(end 131.292893 67.292893)
-		(width 0.25)
+		(width 0.4)
 		(layer "B.Cu")
 		(net 1)
@@
 	)
 	(segment
+		(start 145.775216 65.724784)
+		(end 144.324784 65.724784)
+		(width 0.4)
+		(layer "F.Cu")
+		(net 3)
+	)
+	(segment
 		(start 141.525217 83.275217)
 		(end 137.775216 83.275217)
@@
 	)
 	(segment
+		(start 143.8 65.2)
+		(end 143 66)
+		(width 0.4)
+		(layer "F.Cu")
+		(net 3)
+	)
+	(segment
 		(start 151.125001 78.412499)
 		(end 155.375001 74.162499)
@@
 	)
 	(segment
-		(start 144 65.75)
-		(end 144.025216 65.724784)
-		(width 0.4)
-		(layer "F.Cu")
-		(net 3)
-	)
-	(segment
-		(start 143.974784 65.724784)
-		(end 144 65.75)
-		(width 0.4)
-		(layer "F.Cu")
-		(net 3)
-	)
-	(segment
 		(start 146.224784 83.312716)
 		(end 151.125001 78.412499)
@@
 	)
 	(segment
+		(start 143 66)
+		(end 140.5 66)
+		(width 0.4)
+		(layer "F.Cu")
+		(net 3)
+	)
+	(segment
 		(start 128.225002 68.975002)
 		(end 129 69.75)
@@
 	)
 	(segment
-		(start 144.025216 65.724784)
-		(end 145.775216 65.724784)
-		(width 0.4)
-		(layer "F.Cu")
-		(net 3)
-	)
-	(segment
 		(start 143.000001 86.475002)
 		(end 143.000001 84.749999)
@@
 	)
 	(segment
+		(start 140.5 66)
+		(end 140.224784 65.724784)
+		(width 0.4)
+		(layer "F.Cu")
+		(net 3)
+	)
+	(segment
+		(start 144.324784 65.724784)
+		(end 143.8 65.2)
+		(width 0.4)
+		(layer "F.Cu")
+		(net 3)
+	)
+	(segment
 		(start 134.175432 78.375)
 		(end 134.875 78.375)
@@
 	)
 	(segment
-		(start 140.724782 65.724784)
-		(end 143.974784 65.724784)
-		(width 0.4)
-		(layer "F.Cu")
-		(net 3)
-	)
-	(segment
 		(start 156.074568 74.162499)
 		(end 155.375001 74.162499)
@@
 	)
 	(via
-		(at 144 65.75)
+		(at 143.8 65.2)
 		(size 0.8)
 		(drill 0.4)
@@
 	)
 	(segment
-		(start 143.957107 65.792893)
-		(end 144 65.75)
-		(width 0.4)
-		(layer "B.Cu")
-		(net 3)
-	)
-	(segment
-		(start 132.707107 65.792893)
-		(end 143.957107 65.792893)
+		(start 143 66)
+		(end 132.914214 66)
+		(width 0.4)
+		(layer "B.Cu")
+		(net 3)
+	)
+	(segment
+		(start 143.8 65.2)
+		(end 143 66)
+		(width 0.4)
+		(layer "B.Cu")
+		(net 3)
+	)
+	(segment
+		(start 132.914214 66)
+		(end 132.707107 65.792893)
 		(width 0.4)
 		(layer "B.Cu")
@@
 	)
 	(segment
-		(start 142 64.25)
-		(end 142.025216 64.275216)
+		(start 143.1 64.3)
+		(end 142.2 65.2)
 		(width 0.4)
 		(layer "F.Cu")
@@
 	)
 	(segment
+		(start 143.124784 64.3)
+		(end 143.1 64.3)
+		(width 0.4)
+		(layer "F.Cu")
+		(net 4)
+	)
+	(segment
 		(start 127.475002 71.024998)
 		(end 127.500001 71.024998)
@@
 	)
 	(segment
+		(start 141.275216 64.275216)
+		(end 138.775218 64.275216)
+		(width 0.4)
+		(layer "F.Cu")
+		(net 4)
+	)
+	(segment
 		(start 154.75 60.75)
 		(end 157.224784 63.224784)
@@
 	)
 	(segment
-		(start 138.775218 64.275216)
-		(end 141.974784 64.275216)
-		(width 0.4)
-		(layer "F.Cu")
-		(net 4)
-	)
-	(segment
 		(start 159.75 67.75)
 		(end 157.224784 65.224784)
@@
 	)
 	(segment
-		(start 142.025216 64.275216)
-		(end 147.224784 64.275216)
-		(width 0.4)
-		(layer "F.Cu")
-		(net 4)
-	)
-	(segment
-		(start 141.974784 64.275216)
-		(end 142 64.25)
+		(start 142.2 65.2)
+		(end 141.275216 64.275216)
 		(width 0.4)
 		(layer "F.Cu")
@@
 	)
 	(segment
+		(start 147.224784 64.3)
+		(end 143.124784 64.3)
+		(width 0.4)
+		(layer "F.Cu")
+		(net 4)
+	)
+	(segment
 		(start 138.724783 86.224783)
 		(end 134.974782 82.474782)
@@
 	)
 	(via
-		(at 142 64.25)
+		(at 142.2 65.2)
 		(size 0.8)
 		(drill 0.4)
@@
 	)
 	(segment
-		(start 142 64.25)
-		(end 151.75 64.25)
-		(width 0.4)
-		(layer "B.Cu")
-		(net 4)
-	)
-	(segment
 		(start 153.25 65.75)
 		(end 154.748224 65.75)
@@
 	)
 	(segment
+		(start 151.75 64.25)
+		(end 153.25 65.75)
+		(width 0.4)
+		(layer "B.Cu")
+		(net 4)
+	)
+	(segment
+		(start 143.1 64.3)
+		(end 151.75 64.3)
+		(width 0.4)
+		(layer "B.Cu")
+		(net 4)
+	)
+	(segment
+		(start 143.1 64.3)
+		(end 142.2 65.2)
+		(width 0.4)
+		(layer "B.Cu")
+		(net 4)
+	)
+	(segment
 		(start 154.748224 65.75)
 		(end 155.944544 64.55368)
 		(width 0.4)
 		(layer "B.Cu")
-		(net 4)
-	)
-	(segment
-		(start 151.75 64.25)
-		(end 153.25 65.75)
-		(width 0.4)
-		(layer "B.Cu")

Commit message: Readmes
Changed lines of the file:
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@@
 			)
 		)
+		(property ki_fp_filters "LED* LED_SMD:* LED_THT:*")
+		(sheetname "Root")
+		(sheetfile "heart-badge.kicad_sch")
 		(attr smd)
 		(fp_line
@@
 			)
 		)
+		(property ki_fp_filters "LED* LED_SMD:* LED_THT:*")
+		(sheetname "Root")
+		(sheetfile "heart-badge.kicad_sch")
 		(attr smd)
 		(fp_line
@@
 			)
 		)
+		(property ki_fp_filters "LED* LED_SMD:* LED_THT:*")
+		(sheetname "Root")
+		(sheetfile "heart-badge.kicad_sch")
 		(attr smd)
 		(fp_line
@@
 			)
 		)
+		(property ki_fp_filters "LED* LED_SMD:* LED_THT:*")
+		(sheetname "Root")
+		(sheetfile "heart-badge.kicad_sch")
 		(attr smd)
 		(fp_line
@@
 			)
 		)
+		(property ki_fp_filters "LED* LED_SMD:* LED_THT:*")
+		(sheetname "Root")
+		(sheetfile "heart-badge.kicad_sch")
 		(attr smd)
 		(fp_line
@@
 			)
 		)
+		(property ki_fp_filters "LED* LED_SMD:* LED_THT:*")
+		(sheetname "Root")
+		(sheetfile "heart-badge.kicad_sch")
 		(attr smd)
 		(fp_line
@@
 			)
 		)
+		(property ki_fp_filters "LED* LED_SMD:* LED_THT:*")
+		(sheetname "Root")
+		(sheetfile "heart-badge.kicad_sch")
 		(attr smd)
 		(fp_line
@@
 			)
 		)
+		(property ki_fp_filters "LED* LED_SMD:* LED_THT:*")
+		(sheetname "Root")
+		(sheetfile "heart-badge.kicad_sch")
 		(attr smd)
 		(fp_line
@@
 			)
 		)
+		(property ki_fp_filters "LED* LED_SMD:* LED_THT:*")
+		(sheetname "Root")
+		(sheetfile "heart-badge.kicad_sch")
 		(attr smd)
 		(fp_line
@@
 			)
 		)
+		(property ki_fp_filters "LED* LED_SMD:* LED_THT:*")
+		(sheetname "Root")
+		(sheetfile "heart-badge.kicad_sch")
 		(attr smd)
 		(fp_line
@@
 			)
 		)
+		(property ki_fp_filters "LED* LED_SMD:* LED_THT:*")
+		(sheetname "Root")
+		(sheetfile "heart-badge.kicad_sch")
 		(attr smd)
 		(fp_line
@@
 			)
 		)
+		(property ki_fp_filters "LED* LED_SMD:* LED_THT:*")
+		(sheetname "Root")
+		(sheetfile "heart-badge.kicad_sch")
 		(attr smd)
 		(fp_line
@@
 			)
 		)
+		(property ki_fp_filters "LED* LED_SMD:* LED_THT:*")
+		(sheetname "Root")
+		(sheetfile "heart-badge.kicad_sch")
 		(attr smd)
 		(fp_line
@@
 			)
 		)
+		(property ki_fp_filters "LED* LED_SMD:* LED_THT:*")
+		(sheetname "Root")
+		(sheetfile "heart-badge.kicad_sch")
 		(attr smd)
 		(fp_line
@@
 			)
 		)
+		(property ki_fp_filters "LED* LED_SMD:* LED_THT:*")
+		(sheetname "Root")
+		(sheetfile "heart-badge.kicad_sch")
 		(attr smd)
 		(fp_line
@@
 			)
 		)
+		(property ki_fp_filters "R_*")
+		(sheetname "Root")
+		(sheetfile "heart-badge.kicad_sch")
 		(attr smd)
 		(fp_line
@@
 			)
 		)
+		(sheetname "Root")
+		(sheetfile "heart-badge.kicad_sch")
 		(attr smd)
 		(fp_line
@@
 			)
 		)
+		(sheetname "Root")
+		(sheetfile "heart-badge.kicad_sch")
 		(attr smd)
 		(fp_line
@@
 			(extension_offset 0.5) keep_text_aligned)
 	)
+	(dimension
+		(type aligned)
+		(layer "Cmts.User")
+		(pts
+			(xy 127.467191 62.434264) (xy 150.3 85.267073)
+		)
+		(height 13.241135)
+		(gr_text "32.2905 mm"
+			(at 130.333873 82.400392 315)
+			(layer "Cmts.User")
+			(effects
+				(font
+					(size 1 1)
+					(thickness 0.15)
+				)
+			)
+		)
+		(format
+			(prefix "")
+			(suffix "")
+			(units 3)
+			(units_format 1)
+			(precision 4)
+		)
+		(style
+			(thickness 0.15)
+			(arrow_length 1.27)
+			(text_position_mode 0)
+			(extension_height 0.58642)
+			(extension_offset 0.5) keep_text_aligned)
+	)
+	(dimension
+		(type orthogonal)
+		(layer "Cmts.User")
+		(pts
+			(xy 124.4 69.7) (xy 161.509011 69.713798)
+		)
+		(height -11.9)
+		(orientation 0)
+		(gr_text "37.1090 mm"
+			(at 142.954506 56.65 0)
+			(layer "Cmts.User")
+			(effects
+				(font
+					(size 1 1)
+					(thickness 0.15)
+				)
+			)
+		)
+		(format
+			(prefix "")
+			(suffix "")
+			(units 3)
+			(units_format 1)
+			(precision 4)
+		)
+		(style
+			(thickness 0.15)
+			(arrow_length 1.27)
+			(text_position_mode 0)
+			(extension_height 0.58642)
+			(extension_offset 0.5) keep_text_aligned)
+	)
+	(dimension
+		(type orthogonal)
+		(layer "Cmts.User")
+		(pts
+			(xy 151.268982 59.4) (xy 143.026575 92.2)
+		)
+		(height 12.131018)
+		(orientation 1)
+		(gr_text "32.8000 mm"
+			(at 162.25 75.8 90)
+			(layer "Cmts.User")
+			(effects
+				(font
+					(size 1 1)
+					(thickness 0.15)
+				)
+			)
+		)
+		(format
+			(prefix "")
+			(suffix "")
+			(units 3)
+			(units_format 1)
+			(precision 4)
+		)
+		(style
+			(thickness 0.15)
+			(arrow_length 1.27)
+			(text_position_mode 0)
+			(extension_height 0.58642)
+			(extension_offset 0.5) keep_text_aligned)
+	)
 	(segment
 		(start 131.292893 67.292893)
@@
 		(polygon
 			(pts
-				(xy 122.5 57.5) (xy 162.5 57.5) (xy 162.5 92.5) (xy 122.5 92.5)
+				(xy 103.4 47.65) (xy 189.3 47.65) (xy 189.3 102.05) (xy 103.4 102.05)
 			)
 		)

Commit message: Heart
Parts:
- moved R1 0.50 mm to (132.0, 67.0)
- moved SW1 0.35 mm to (154.2, 66.8)
Routing:
- net Net-(D1-K): track 122.3 -> 109.9 mm
- net Net-(D1-A): track 142.4 -> 134.3 mm
Other:
- board text added: "pajecistavebnice.cz"
- board text removed: "github.com/polaracep"
