File: mddm-badge/pcb/mddm-badge-tooling.kicad_pcb (KiCad board)
At the start: 2 copper layers, 26.8 x 31.4 mm, 20 parts, among them J1 Conn_01x06, SW1 SKRKAEE020, U1 PIC10F322-IOT

Commit message: Bat V2.1, mddm-badge tooling added
Parts:
- added REF**: jlc_hole, lib:jlc_hole, F.Cu at (156.2, 108.4)
- added REF**: jlc_hole, lib:jlc_hole, F.Cu at (136.8, 108.4)
- J1: value Conn_01x06 -> Conn_01x05
Routing:
- net /button: track 30.2 -> 27.0 mm
- net /blue: track 88.9 -> 85.8 mm
- net GND: track 41.1 -> 40.5 mm
Other:
- board text added: "<- TOOLING HOLE"
- board text added: "TOOLING HOLE ->"
