File: crossing/crossing-blink/crossing.kicad_pcb (KiCad board)
At the start: 2 copper layers, 38 x 66.8 mm, 18 parts, among them Q1 2N3904, Q2 2N3904, Q3 2N3904, Q4 2N3904, SW1 SW_SPDT

Commit message: Some updates, added new library symbols/fps.
Parts:
- turned H1 to 15 degrees
